Commit message: spot walked initially

File: spot_description/models/spot/model.urdf (robot description, URDF)
Before this commit: robot spot, 27 links, 26 joints
Links:
- removed link battery
- removed link camera_back
- removed link camera_frontleft
- removed link camera_frontright
- removed link camera_left
- removed link camera_right
- removed link imu
- link base_link: mass 20.492 -> 16.0; geometry collision mesh filename=file:///root/spot_ws/install/spot_description/share/spot_de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; visual mesh filename=file:///root/spot_ws/install/spot_description/share/spot_de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
- link body: mass 1e-05 -> None
- link front_left_ee: mass 1e-05 -> None
- link front_left_hip: mass 2 -> 2.0; geometry collision mesh filename=file:///root/spot_ws/install/spot_description/share/spot_de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; visual mesh filename=file:///root/spot_ws/install/spot_description/share/spot_de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
- link front_left_lower_leg: geometry collision mesh filename=file:///root/spot_ws/install/spot_description/share/spot_de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 scale=-1.82 0.97 0.98; visual mesh filename=file:///root/spot_ws/install/spot_description/share/spot_de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
- link front_left_upper_leg: mass 1 -> 1.0; geometry collision mesh filename=file:///root/spot_ws/install/spot_description/share/spot_de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; visual mesh filename=file:///root/spot_ws/install/spot_description/share/spot_de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
- link front_rail: mass 1e-05 -> None
- link front_right_ee: mass 1e-05 -> None
- link front_right_hip: mass 2 -> 2.0; geometry collision mesh filename=file:///root/spot_ws/install/spot_description/share/spot_de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; visual mesh filename=file:///root/spot_ws/install/spot_description/share/spot_de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
- link front_right_lower_leg: geometry collision mesh filename=file:///root/spot_ws/install/spot_description/share/spot_de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 scale=-1.82 0.97 0.98; visual mesh filename=file:///root/spot_ws/install/spot_description/share/spot_de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
- link front_right_upper_leg: mass 1 -> 1.0; geometry collision mesh filename=file:///root/spot_ws/install/spot_description/share/spot_de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; visual mesh filename=file:///root/spot_ws/install/spot_description/share/spot_de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
- link rear_left_ee: mass 1e-05 -> None
- link rear_left_hip: mass 2 -> 2.0; geometry collision mesh filename=file:///root/spot_ws/install/spot_description/share/spot_de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; visual mesh filename=file:///root/spot_ws/install/spot_description/share/spot_de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
- link rear_left_lower_leg: geometry collision mesh filename=file:///root/spot_ws/install/spot_description/share/spot_de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 scale=-1.82 0.97 0.98; visual mesh filename=file:///root/spot_ws/install/spot_description/share/spot_de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
- link rear_left_upper_leg: mass 1 -> 1.0; geometry collision mesh filename=file:///root/spot_ws/install/spot_description/share/spot_de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; visual mesh filename=file:///root/spot_ws/install/spot_description/share/spot_de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
- link rear_rail: mass 1e-05 -> None
- link rear_right_ee: mass 1e-05 -> None
- link rear_right_hip: mass 2 -> 2.0; geometry collision mesh filename=file:///root/spot_ws/install/spot_description/share/spot_de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; visual mesh filename=file:///root/spot_ws/install/spot_description/share/spot_de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
- link rear_right_lower_leg: geometry collision mesh filename=file:///root/spot_ws/install/spot_description/share/spot_de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 scale=-1.82 0.97 0.98; visual mesh filename=file:///root/spot_ws/install/spot_description/share/spot_de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
- link rear_right_upper_leg: mass 1 -> 1.0; geometry collision mesh filename=file:///root/spot_ws/install/spot_description/share/spot_de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; visual mesh filename=file:///root/spot_ws/install/spot_description/share/spot_de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
Joints:
- removed joint battery_joint
- removed joint camera_back_j
- removed joint camera_frontleft_j
- removed joint camera_frontright_j
- removed joint camera_left_j
- removed joint camera_right_j
- removed joint imu_j
- joint base_link_joint: origin xyz=0 0 1 -> xyz=0 0 0 rpy=0 0 0
- joint front_left_foot: origin xyz=0 0 1 -> xyz=0 0 -0.37 rpy=0 0 0
- joint front_left_hip_x: limit lower=-0.785398 upper=0.785398 effort=80 velocity=15 -> lower=-0.78539816339744827899 upper=0.78539816339744827899 effort=100 velocity=1000.00; origin xyz=1 0 0 -> xyz=0.29785 0.055 0 rpy=0 0 0; parent base_link -> body
- joint front_left_hip_y: limit lower=-0.898845 upper=2.29511 effort=80 velocity=15 -> lower=-0.89884456477707963539 upper=2.2951079663725435509 effort=100 velocity=1000.00; origin xyz=0 1 0 -> xyz=0 0.110945 0 rpy=0 0 0
- joint front_left_knee: limit lower=-2.7929 upper=-0.254801 effort=80 velocity=15 -> lower=-2.7929 upper=-0.254801 effort=100 velocity=1000.00; origin xyz=0 1 0 -> xyz=0.025 0 -0.3205 rpy=0 0 0
- joint front_rail_joint: origin xyz=0 0 1 -> xyz=0.223 0 0.0805 rpy=0 0 0; parent body -> base_link
- joint front_right_foot: origin xyz=0 0 1 -> xyz=0 0 -0.37 rpy=0 0 0
- joint front_right_hip_x: limit lower=-0.785398 upper=0.785398 effort=80 velocity=15 -> lower=-0.78539816339744827899 upper=0.78539816339744827899 effort=100 velocity=1000.00; origin xyz=1 0 0 -> xyz=0.29785 -0.055 0 rpy=0 0 0; parent base_link -> body
- joint front_right_hip_y: limit lower=-0.898845 upper=2.29511 effort=80 velocity=15 -> lower=-0.89884456477707963539 upper=2.2951079663725435509 effort=100 velocity=1000.00; origin xyz=0 1 0 -> xyz=0 -0.110945 0 rpy=0 0 0
- joint front_right_knee: limit lower=-2.7929 upper=-0.254801 effort=80 velocity=15 -> lower=-2.7929 upper=-0.254801 effort=100 velocity=1000.00; origin xyz=0 1 0 -> xyz=0.025 0 -0.3205 rpy=0 0 0
- joint rear_left_foot: origin xyz=0 0 1 -> xyz=0 0 -0.37 rpy=0 0 0
- joint rear_left_hip_x: limit lower=-0.785398 upper=0.785398 effort=80 velocity=15 -> lower=-0.78539816339744827899 upper=0.78539816339744827899 effort=100 velocity=1000.00; origin xyz=1 0 0 -> xyz=-0.29785 0.055 0 rpy=0 0 0; parent base_link -> body
- joint rear_left_hip_y: limit lower=-0.898845 upper=2.29511 effort=80 velocity=15 -> lower=-0.89884456477707963539 upper=2.2951079663725435509 effort=100 velocity=1000.00; origin xyz=0 1 0 -> xyz=0 0.110945 0 rpy=0 0 0
- joint rear_left_knee: limit lower=-2.7929 upper=-0.254801 effort=80 velocity=15 -> lower=-2.7929 upper=-0.254801 effort=100 velocity=1000.00; origin xyz=0 1 0 -> xyz=0.025 0 -0.3205 rpy=0 0 0
- joint rear_rail_joint: origin xyz=0 0 1 -> xyz=-0.223 0 0.0805 rpy=0 0 0; parent body -> base_link
- joint rear_right_foot: origin xyz=0 0 1 -> xyz=0 0 -0.37 rpy=0 0 0
- joint rear_right_hip_x: limit lower=-0.785398 upper=0.785398 effort=80 velocity=15 -> lower=-0.78539816339744827899 upper=0.78539816339744827899 effort=100 velocity=1000.00; origin xyz=1 0 0 -> xyz=-0.29785 -0.055 0 rpy=0 0 0; parent base_link -> body
- joint rear_right_hip_y: limit lower=-0.898845 upper=2.29511 effort=80 velocity=15 -> lower=-0.89884456477707963539 upper=2.2951079663725435509 effort=100 velocity=1000.00; origin xyz=0 1 0 -> xyz=0 -0.110945 0 rpy=0 0 0
- joint rear_right_knee: limit lower=-2.7929 upper=-0.254801 effort=80 velocity=15 -> lower=-2.7929 upper=-0.254801 effort=100 velocity=1000.00; origin xyz=0 1 0 -> xyz=0.025 0 -0.3205 rpy=0 0 0

Commit message: move the meshes and change urdf file paths

File: spot_description/models/spot/model.urdf (robot description, URDF)
Before this commit: robot spot, 20 links, 19 joints
Links:
- link base_link: geometry collision mesh filename=package://spot_description/meshes/body_collision.stl; visual mesh filename=package://spot_description/meshes/body.dae
- link front_left_hip: geometry collision mesh filename=package://spot_description/meshes/front_left_hip_collision.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; visual mesh filename=package://spot_description/meshes/front_left_hip.dae
- link front_left_lower_leg: geometry collision mesh filename=package://spot_description/meshes/front_left_lower_leg_coll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 scale=-1.82 0.97 0.98; visual mesh filename=package://spot_description/meshes/front_left_lower_leg.dae
- link front_left_upper_leg: geometry collision mesh filename=package://spot_description/meshes/front_left_upper_leg_coll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; visual mesh filename=package://spot_description/meshes/front_left_upper_leg.dae
- link front_right_hip: geometry collision mesh filename=package://spot_description/meshes/front_right_hip_collision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; visual mesh filename=package://spot_description/meshes/front_right_hip.dae
- link front_right_lower_leg: geometry collision mesh filename=package://spot_description/meshes/front_right_lower_leg_col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 scale=-1.82 0.97 0.98; visual mesh filename=package://spot_description/meshes/front_right_lower_leg.dae
- link front_right_upper_leg: geometry collision mesh filename=package://spot_description/meshes/front_right_upper_leg_col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; visual mesh filename=package://spot_description/meshes/front_right_upper_leg.dae
- link rear_left_hip: geometry collision mesh filename=package://spot_description/meshes/rear_left_hip_collision.s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; visual mesh filename=package://spot_description/meshes/rear_left_hip.dae
- link rear_left_lower_leg: geometry collision mesh filename=package://spot_description/meshes/rear_left_lower_leg_colli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 scale=-1.82 0.97 0.98; visual mesh filename=package://spot_description/meshes/rear_left_lower_leg.dae
- link rear_left_upper_leg: geometry collision mesh filename=package://spot_description/meshes/rear_left_upper_leg_colli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; visual mesh filename=package://spot_description/meshes/rear_left_upper_leg.dae
- link rear_right_hip: geometry collision mesh filename=package://spot_description/meshes/rear_right_hip_collision.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; visual mesh filename=package://spot_description/meshes/rear_right_hip.dae
- link rear_right_lower_leg: geometry collision mesh filename=package://spot_description/meshes/rear_right_lower_leg_coll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 scale=-1.82 0.97 0.98; visual mesh filename=package://spot_description/meshes/rear_right_lower_leg.dae
- link rear_right_upper_leg: geometry collision mesh filename=package://spot_description/meshes/rear_right_upper_leg_coll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; visual mesh filename=package://spot_description/meshes/rear_right_upper_leg.dae
